Commit message: Added Visualization for ros package with dmoc and reconfiguration ability using a gui for gcop_ctrl.

File: ros_packages/gcop_urdf/rccar.urdf (robot description, URDF)
Before this commit: robot Unicycle, 5 links, 4 joints
Links:
- link backwheel1: geometry visual cylinder length=0.04 radius=0.04
- link backwheel2: geometry visual cylinder length=0.04 radius=0.04
Joints:
- removed joint frontwheel1_to_frontwheel2
- added joint base_to_frontwheel2: type continuous, parent carbody, child frontwheel2, origin xyz=0.10 0.07 0 rpy=-1.5707 0 0, axis 0 -1 0
- joint backwheel1_to_backwheel2: origin xyz=0 0 0.16 rpy=0 0 0 -> xyz=0 0 0.14 rpy=0 0 0
- joint base_to_backwheel1: origin xyz=-0.15 -0.08 0 rpy=-1.5707 0 0 -> xyz=-0.15 -0.07 0 rpy=-1.5707 0 0
- joint base_to_frontwheel1: axis 0 0 1 -> 0 -1 0

Commit message: Added car model and working controller for the car

File: ros_packages/gcop_urdf/rccar.urdf (robot description, URDF)
Before this commit: robot Unicycle, 5 links, 4 joints
Links:
- added link baselink
- added link kinect; visual mesh filename=package://gcop_urdf/meshes/kinect_sensor.dae scale=0.00001 0.00001 0.00001
- link carbody: geometry visual mesh filename=package://gcop_urdf/meshes/carwithoutfronttyres.dae scale=0.001 0.001 0.001
Joints:
- added joint basetocarbody: type fixed, parent baselink, child carbody, origin xyz=0.15 0.0 0 rpy=0 0 0
- added joint carbodytokinect: type fixed, parent carbody, child kinect, origin xyz=0.15 0.0 0 rpy=0 0 0
- joint backwheel1_to_backwheel2: origin xyz=0 0 0.14 rpy=0 0 0 -> xyz=0 0 0.260 rpy=0 0 0
- joint base_to_backwheel1: origin xyz=-0.15 -0.07 0 rpy=-1.5707 0 0 -> xyz=-0.15 -0.13 0 rpy=-1.5707 0 0
- joint base_to_frontwheel1: origin xyz=0.10 -0.07 0 rpy=-1.5707 0 0 -> xyz=0.15 -0.14 0 rpy=-1.5707 0 0
- joint base_to_frontwheel2: origin xyz=0.10 0.07 0 rpy=-1.5707 0 0 -> xyz=0.15 0.14 0 rpy=-1.5707 0 0

Commit message: Added header files from ros urdf

File: ros_packages/gcop_urdf/rccar.urdf (robot description, URDF)
Before this commit: robot Unicycle, 7 links, 6 joints
Links:
- link carbody: mass None -> 10
