Commit message: More visualization stuff

File: ros_packages/gcop_urdf/chain.urdf (robot description, URDF)
Before this commit: robot Chain, 6 links, 5 joints
Joints:
- joint link1tolink3: origin xyz=0.05 0.0 0 rpy=0 0 0 -> xyz=0.1 0.0 0 rpy=0 0 0
- joint link2tolink4: origin xyz=-0.05 0.0 0 rpy=0 0 0 -> xyz=-0.1 0.0 0 rpy=0 0 0
- joint roottolink1: origin xyz=0.15 0.0 0 rpy=0 0 0 -> xyz=0.2 0.0 0 rpy=0 0 0
- joint roottolink2: origin xyz=-0.15 0.0 0 rpy=0 0 0 -> xyz=-0.2 0.0 0 rpy=0 0 0

Commit message: intermediate commit to show completion of ctrltrajpublishing for general bodies

File: ros_packages/gcop_urdf/chain.urdf (robot description, URDF)
Before this commit: robot Chain, 6 links, 5 joints
Joints:
- joint roottolink1: origin xyz=0.2 0.0 0 rpy=0 0 0 -> xyz=0.15 0.0 0 rpy=0 0 0
- joint roottolink2: origin xyz=-0.2 0.0 0 rpy=0 0 0 -> xyz=-0.15 0.0 0 rpy=0 0 0

Commit message: Added working chain dynamics simulator and visualizer

File: ros_packages/gcop_urdf/chain.urdf (robot description, URDF)
Before this commit: robot Chain, 6 links, 5 joints
Links:
- removed link link3
- removed link link4
Joints:
- removed joint link1tolink3
- removed joint link2tolink4
- joint roottolink1: limit lower=-2.2 upper=0.7 effort=30 velocity=1.0 -> lower=-5 upper=5 effort=30 velocity=5.0
- joint roottolink2: limit lower=-2.2 upper=0.7 effort=30 velocity=1.0 -> lower=-5 upper=5 effort=30 velocity=5.0
