Commit message: added lots of working mbs systems as urdf files completed stage 1 of integrating ros with mbs in the form of urdf files

File: ros_packages/gcop_ctrl/params/airbot.urdf (robot description, URDF)
Before this commit: robot Airbot, 4 links, 3 joints
Links:
- link airbase: geometry visual box size=0.3 0.1 0.05
Joints:
- removed joint basetoroot
- removed joint roottolink1
- removed joint roottolink2
- added joint airbasetolink1: type revolute, parent airbase, child link1, origin xyz=0.15 0.0 0 rpy=0 0 0, axis 0 -1 0, limit lower=-5 upper=5 effort=30 velocity=5.0
- added joint airbasetolink2: type revolute, parent airbase, child link2, origin xyz=-0.15 0.0 0 rpy=0 0 0, axis 0 -1 0, limit lower=-5 upper=5 effort=30 velocity=5.0
- added joint basetoairbase: type fixed, parent baselink, child airbase, origin xyz=0 0 0 rpy=0 0 0

File: ros_packages/gcop_ctrl/params/chain1.urdf (robot description, URDF)
Before this commit: robot Chain, 4 links, 3 joints
Links:
- removed link root
- added link chainbase, mass 3; visual box size=0.3 .10 0.05
Joints:
- joint basetoroot: child root -> chainbase
- joint roottolink1: parent root -> chainbase
- joint roottolink2: parent root -> chainbase
