Commit message: fixed a bug in urdfparsing algorithm for fixed joints and added support for the new integrator and dynamics of urdf files

File: ros_packages/gcop_ctrl/params/airbot2.urdf (robot description, URDF)
Before this commit: robot Chain, 6 links, 5 joints
Joints:
- joint airbasetolink1: limit lower=-2.2 upper=0.7 effort=30 velocity=1.0 -> lower=-3.14 upper=3.14 effort=30 velocity=1.0
- joint airbasetolink2: limit lower=-2.2 upper=0.7 effort=30 velocity=1.0 -> lower=-3.14 upper=3.14 effort=30 velocity=1.0
- joint link1tolink3: limit lower=-2.2 upper=0.7 effort=30 velocity=1.0 -> lower=-3.14 upper=3.14 effort=30 velocity=1.0
- joint link2tolink4: limit lower=-2.2 upper=0.7 effort=30 velocity=1.0 -> lower=-3.14 upper=3.14 effort=30 velocity=1.0

File: ros_packages/gcop_ctrl/params/airbot3.urdf (robot description, URDF)
Before this commit: robot Airbot, 8 links, 7 joints
Joints:
- joint airbasetolink1: limit lower=-5 upper=5 effort=30 velocity=5.0 -> lower=-3.14 upper=3.14 effort=30 velocity=10.0
- joint airbasetolink4: limit lower=-5 upper=5 effort=30 velocity=5.0 -> lower=-3.14 upper=3.14 effort=30 velocity=10.0
- joint link1tolink2: limit lower=-5 upper=5 effort=30 velocity=5.0 -> lower=-3.14 upper=3.14 effort=30 velocity=10.0
- joint link2tolink3: limit lower=-5 upper=5 effort=30 velocity=5.0 -> lower=-3.14 upper=3.14 effort=30 velocity=10.0
- joint link4tolink5: limit lower=-5 upper=5 effort=30 velocity=5.0 -> lower=-3.14 upper=3.14 effort=30 velocity=10.0
- joint link5tolink6: limit lower=-5 upper=5 effort=30 velocity=5.0 -> lower=-3.14 upper=3.14 effort=30 velocity=10.0

File: ros_packages/gcop_ctrl/params/airbot3.xacro (robot description, xacro)
@@ -7,5 +7,5 @@
 <xacro:property name="l3" value=".3" />
 <!--Structural Properties-->
-<xacro:property name="m0" value="3" />
+<xacro:property name="m0" value="1" />
 <xacro:property name="m1" value=".2" />
 <xacro:property name="m2" value=".3" />
@@ -128,5 +128,5 @@
 		<origin rpy="0 0 0" xyz="0 ${y0} ${-z0}"/>
     <axis xyz="0 0 1"/>
-		<limit effort="30" velocity="5.0" lower="-5" upper="5" />
+		<limit effort="30" velocity="10.0" lower="-3.14" upper="3.14" />
   </joint>
 	<joint name="link1tolink2" type="revolute">
@@ -135,5 +135,5 @@
 		<origin rpy="0 0 0" xyz="0 ${l1} 0"/>
     <axis xyz="0 1 0"/>
-		<limit effort="30" velocity="5.0" lower="-5" upper="5" />
+		<limit effort="30" velocity="10.0" lower="-3.14" upper="3.14" />
   </joint>
 	<joint name="link2tolink3" type="revolute">
@@ -142,5 +142,5 @@
 		<origin rpy="0 0 0" xyz="0 0 ${-l2}"/>
     <axis xyz="0 1 0"/>
-		<limit effort="30" velocity="5.0" lower="-5" upper="5" />
+		<limit effort="30" velocity="10.0" lower="-3.14" upper="3.14" />
   </joint>
   <joint name="airbasetolink4" type="revolute">
@@ -149,5 +149,5 @@
 		<origin rpy="0 0 0" xyz="0 ${-y0} ${-z0}"/>
     <axis xyz="0 0 1"/>
-		<limit effort="30" velocity="5.0" lower="-5" upper="5" />
+		<limit effort="30" velocity="10.0" lower="-3.14" upper="3.14" />
   </joint>
 	<joint name="link4tolink5" type="revolute">
@@ -156,5 +156,5 @@
 		<origin rpy="0 0 0" xyz="0 ${-l1} 0"/>
     <axis xyz="0 1 0"/>
-		<limit effort="30" velocity="5.0" lower="-5" upper="5" />
+		<limit effort="30" velocity="10.0" lower="-3.14" upper="3.14" />
   </joint>
 	<joint name="link5tolink6" type="revolute">
@@ -163,5 +163,5 @@
 		<origin rpy="0 0 0" xyz="0 0 ${-l2}"/>
     <axis xyz="0 1 0"/>
-		<limit effort="30" velocity="5.0" lower="-5" upper="5" />
+		<limit effort="30" velocity="10.0" lower="-3.14" upper="3.14" />
   </joint>
 </robot>

File: ros_packages/gcop_ctrl/params/airbot4.urdf (robot description, URDF)
Before this commit: robot Airbot, 8 links, 7 joints
Joints:
- joint airbasetolink1: limit lower=-5 upper=5 effort=30 velocity=5.0 -> lower=-3.14 upper=3.14 effort=30 velocity=10.0
- joint airbasetolink4: limit lower=-5 upper=5 effort=30 velocity=5.0 -> lower=-3.14 upper=3.14 effort=30 velocity=10.0
- joint link1tolink2: limit lower=-5 upper=5 effort=30 velocity=5.0 -> lower=-3.14 upper=3.14 effort=30 velocity=10.0
- joint link2tolink3: limit lower=-5 upper=5 effort=30 velocity=5.0 -> lower=-3.14 upper=3.14 effort=30 velocity=10.0
- joint link4tolink5: limit lower=-5 upper=5 effort=30 velocity=5.0 -> lower=-3.14 upper=3.14 effort=30 velocity=10.0
- joint link5tolink6: limit lower=-5 upper=5 effort=30 velocity=5.0 -> lower=-3.14 upper=3.14 effort=30 velocity=10.0

File: ros_packages/gcop_ctrl/params/airbot4.xacro (robot description, xacro)
@@ -133,5 +133,5 @@
 		<origin rpy="0 0 0" xyz="0 ${y0} ${-z0}"/>
     <axis xyz="0 0 1"/>
-		<limit effort="30" velocity="5.0" lower="-5" upper="5" />
+		<limit effort="30" velocity="10.0" lower="-3.14" upper="3.14" />
   </joint>
 	<joint name="link1tolink2" type="revolute">
@@ -140,5 +140,5 @@
 		<origin rpy="0 0 0" xyz="0 ${l1} 0"/>
     <axis xyz="0 1 0"/>
-		<limit effort="30" velocity="5.0" lower="-5" upper="5" />
+		<limit effort="30" velocity="10.0" lower="-3.14" upper="3.14" />
   </joint>
 	<joint name="link2tolink3" type="revolute">
@@ -147,5 +147,5 @@
 		<origin rpy="0 0 0" xyz="0 0 ${-l2}"/>
     <axis xyz="0 1 0"/>
-		<limit effort="30" velocity="5.0" lower="-5" upper="5" />
+		<limit effort="30" velocity="10.0" lower="-3.14" upper="3.14" />
   </joint>
   <joint name="airbasetolink4" type="revolute">
@@ -154,5 +154,5 @@
 		<origin rpy="0 0 0" xyz="0 ${-y0} ${-z0}"/>
     <axis xyz="0 0 1"/>
-		<limit effort="30" velocity="5.0" lower="-5" upper="5" />
+		<limit effort="30" velocity="10.0" lower="-3.14" upper="3.14" />
   </joint>
 	<joint name="link4tolink5" type="revolute">
@@ -161,5 +161,5 @@
 		<origin rpy="0 0 0" xyz="0 ${-l1} 0"/>
     <axis xyz="0 1 0"/>
-		<limit effort="30" velocity="5.0" lower="-5" upper="5" />
+		<limit effort="30" velocity="10.0" lower="-3.14" upper="3.14" />
   </joint>
 	<joint name="link5tolink6" type="revolute">
@@ -168,5 +168,5 @@
 		<origin rpy="0 0 0" xyz="0 0 ${-l2}"/>
     <axis xyz="0 1 0"/>
-		<limit effort="30" velocity="5.0" lower="-5" upper="5" />
+		<limit effort="30" velocity="10.0" lower="-3.14" upper="3.14" />
   </joint>
 </robot>

File: ros_packages/gcop_ctrl/params/chain1.urdf (robot description, URDF)
Before this commit: robot Chain, 4 links, 3 joints
Joints:
- joint roottolink1: limit lower=-5 upper=5 effort=30 velocity=5.0 -> lower=-3.14 upper=3.14 effort=30 velocity=5.0
- joint roottolink2: limit lower=-5 upper=5 effort=30 velocity=5.0 -> lower=-3.14 upper=3.14 effort=30 velocity=5.0

File: ros_packages/gcop_ctrl/params/chain2_2.urdf (robot description, URDF)
Before this commit: robot Chain, 6 links, 5 joints
Joints:
- removed joint link1tolink3
- removed joint link2tolink4
- removed joint roottolink2
- added joint link1tolink2: type revolute, parent link1, child link2, origin xyz=0.1 0.0 0 rpy=0 0 0, axis 0 -1 0, limit lower=-2.2 upper=0.7 effort=30 velocity=1.0
- added joint link2tolink3: type revolute, parent link2, child link3, origin xyz=0.1 0.0 0 rpy=0 0 0, axis 0 -1 0, limit lower=-2.2 upper=0.7 effort=30 velocity=1.0
- added joint link3tolink4: type revolute, parent link3, child link4, origin xyz=0.1 0.0 0 rpy=0 0 0, axis 0 -1 0, limit lower=-2.2 upper=0.7 effort=30 velocity=1.0
- joint roottolink1: limit lower=-3.14 upper=3.14 effort=30 velocity=1.0 -> lower=-2.2 upper=0.7 effort=30 velocity=1.0

File: ros_packages/gcop_ctrl/params/chain3.urdf (robot description, URDF)
Before this commit: robot Chain, 6 links, 5 joints
Links:
- added link link4, mass 1; visual box size=0.1 0.05 0.1
Joints:
- added joint link3tolink4: type revolute, parent link3, child link4, origin xyz=0.0 0.0 0.05 rpy=0 0 0, axis 0 -1 0, limit lower=-5 upper=5 effort=30 velocity=5.0
- joint fixedlinktolink3: axis 0 -1 0 -> (none); limit lower=-5 upper=5 effort=30 velocity=5.0 -> (none); type revolute -> fixed

File: ros_packages/gcop_ctrl/params/chain3.xacro (robot description, xacro)
@@ -63,4 +63,19 @@
         <box size="0.1 0.05 0.1"/>
       </geometry>
+      <material name="red">
+        <color rgba="0.8 0 0 1"/>
+      </material>
+    </visual>
+    <inertial>
+			<origin rpy="0 0 0" xyz="0.0 0.0 0.05"/>
+			<xacro:compute_inertia mass="${m}" x="0.1" y="0.05" z="0.1"/>
+    </inertial>
+  </link>
+	<link name="link4">
+    <visual>
+			<origin rpy="0 0 0" xyz="0.0 0.0 0.05"/>
+      <geometry>
+        <box size="0.1 0.05 0.1"/>
+      </geometry>
       <material name="blue">
         <color rgba="0 0 0.8 1"/>
@@ -83,7 +98,12 @@
     <origin rpy="0 0 0" xyz="0.0 0.0 0.1"/>
   </joint>
-	<joint name="fixedlinktolink3" type="revolute">
+	<joint name="fixedlinktolink3" type="fixed">
     <parent link="fixedlink"/>
     <child link="link3"/>
+    <origin rpy="0 0 0" xyz="0.0 0.0 0.05"/>
+  </joint>
+	<joint name="link3tolink4" type="revolute">
+    <parent link="link3"/>
+    <child link="link4"/>
     <origin rpy="0 0 0" xyz="0.0 0.0 0.05"/>
     <axis xyz="0 -1 0"/>
