Commit message: Added Multiple robots for rviz and tried debugging problems

File: ros_packages/gcop_ctrl/params/chain1_3.urdf (robot description, URDF)
Before this commit: robot Chain, 4 links, 3 joints
Links:
- link chainbase: mass 3 -> 0.0001
- link link1: mass 1 -> 5.70044; geometry visual box size=0.1 0.1 0.05
- link link2: mass 1 -> 3.22698; geometry visual box size=0.1 0.1 0.05
Joints:
- removed joint roottolink2
- added joint link1tolink2: type revolute, parent link1, child link2, origin xyz=0.1 0 0.0 rpy=-1.57079632679 0 0, axis 0 0 1, limit lower=-2.147 upper=1.047 effort=100 velocity=1.5
- joint roottolink1: axis 0 -1 0 -> 0 0 1; limit lower=-5 upper=5 effort=30 velocity=5.0 -> lower=-1.7 upper=1.7 effort=100 velocity=1.5; origin xyz=0.15 0.0 0 rpy=0 0 0 -> xyz=0.0 0.0 0 rpy=0 0 0
